File: Electronic_load_PCB/Electronic_load.brd (EAGLE design)
At the start: 121.9 x 88.6 mm, 109 parts, among them IC7 LM1117IMPX-5.0, J1 XT60-M, J2 B2B-XH, J3 B4B-XH, J4 B2B-XH, J5 B2B-XH, J6 B2B-XH, J7 B2B-XH, Q1 IRFP250, Q10 S9015, Q11 S9015, Q12 CRYSTAL_3,4X2,7, Q2 IRFP250, Q3 IRFP250, Q4 IRFP250, Q5 32768Hz, Q6 IRLML6244, Q7 BD911, Q8 S9015, Q9 S9015, U1 ANALOG_DEVICES_AD8630ARZ-REEL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, U2 MCP4725A0T-E/CH, U3 ADS1115, U4 ATMEGA328P-AU, U5 OPA277-SOIC08, U6 MCP79410-I/SN, U7 ICL7660CPAZSOIC, U8 PC817X2NIP0F

Commit message: finished V1.0
Parts:
- added J8: B5B-XH, jst connectors:JST_B5B-XH-A(LF)(SN)
- added R29: 10k, rcl:R0603
- C6: value (none) -> 100n
- JP2: value (none) -> B4B-XH; device pinhead:1X04 -> jst connectors:JST_B4B-XH-A(LF)(SN)
- R27, R28: value (none) -> 4k7
- moved JP2 16.5 mm to (114.9, 45.1)
- moved C14 0.64 mm to (103.5, 43.1)
- moved C15 0.64 mm to (103.5, 41.0)
- moved Q5 0.64 mm to (107.3, 41.7)
- moved U6 0.64 mm to (106.0, 36.2)
- moved C16 0.63 mm to (109.9, 34.9)
- moved J6 0.13 mm to (115.4, 18.4)
Connections:
- new net ENC_A: J8.3, U4.32
- new net ENC_B: J8.2, U4.26
- new net ENC_SW: J8.4, U4.1
- net 5V: now also J8.1, R29.1
- net GND: now also J8.5
- net RST: now also R29.2
- net TRIGG: now also U4.22
Routing:
- net ENC_SW: track 0.00 -> 30.4 mm
- net ENC_A: track 0.00 -> 25.4 mm
- net TRIGG: track 2.91 -> 24.6 mm, vias 0 -> 2
- net RST: track 32.3 -> 51.0 mm
- net ENC_B: track 0.00 -> 17.8 mm
- net TX: track 24.4 -> 40.3 mm
- net RX: track 21.5 -> 37.1 mm
- net GND: track 497.9 -> 511.6 mm, vias 156 -> 159
- net 12V: track 61.9 -> 64.6 mm
- net 4,096V: track 33.6 -> 32.0 mm
- net SCL: track 71.5 -> 71.2 mm, vias 4 -> 6
- net 5V: track 278.0 -> 278.3 mm, vias 70 -> 68
- net SDA: track 64.3 -> 64.1 mm, vias 2 -> 4
Other:
- outline, holes or cut-outs redrawn
- board text added: "10k NTC"
- board text added: "GND"
- board text added: "Keypad"
- board text added: "RST"
- board text added: "RX"
- board text added: "Rotary encoder"
- board text added: "TX"
