File: Electronic_load_PCB/Electronic_load.sch (EAGLE design)
At the start: 70 parts, among them IC2 7805TV, J1 XT60-M, Q1 IRFP250, Q2 IRFP250, Q3 IRFP250, Q4 IRFP250, U1 ANALOG_DEVICES_AD8630ARZ-REEL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, U2 MCP4725A0T-E/CH, U3 ADS1115, U4 ATMEGA328P-AU, U5 OPA277-SOIC08, U6 MCP79410-I/SN, U7 ICL7660CPAZ

Commit message: Power supply schematic done
Parts:
- removed B1: (no value), rectifier:FB15
- removed IC2: 7805TV, linear:7805TV
- removed SJ1: (no value), jumper:SJ
- removed X1: (no value), con-wago-500:W237-102
- added C21, C22: 100n, rcl:C-EUC0603
- added C23: 100n, rcl:C-EUC0603K
- added C24: 10u, rcl:CPOL-EUCT3528
- added C25: 1u, rcl:C-EUC0603
- added C26, C27: 10u, rcl:CPOL-EUB/3528-21W
- added D1, D2, D3, D4: 1N5819-B, diode:1N5819-B
- added IC7: LM1117IMPX-5.0, lm1117:LM1117IMPX-5.0
- added J3: B4B-XH-A(LF)(SN), B4B-XH-A_LF__SN_:B4B-XH-A(LF)(SN)
- added J4, J5: B2B-XH-A(LF)(SN), JST_B2B-XH-A_LF__SN_:B2B-XH-A(LF)(SN)
- added Q6: IRLML6244, IRLML6244:IRLML6244
- added Q7: BD911, BD911:BD911
- added R30: (no value), rcl:R-EU_R0603
- added R31: 1R, rcl:R-EU_R0805
- added R32, R33: 1R, rcl:R-EU_R0603
- added SPI: (no value), con-lstb:MA03-2
- added U$3: BYG22B, BYG22B:BYG22B
- added VR1: (no value), tl431:TL431CLP
- C11, C12: value (none) -> 4700u; device rcl:CPOL-EUE10-20 -> rcl:CPOL-EUE7.5-16
- C14, C15: value (none) -> 6-9p
- C17, C18: value 10u -> 100u
- J2: value (none) -> B2B-XH-A(LF)(SN); device con-amp:MTA02-156 -> JST_B2B-XH-A_LF__SN_:B2B-XH-A(LF)(SN)
- KK2: value SK104-PAD -> SK95-2M3; device heatsink:SK104-PAD -> heatsink:SK95-2M3
- R1, R11, R16, R6: value 100 -> 1k; device rcl:R-EU_R0603 -> rcl:R-EU_R0805
- R10, R14, R15, R19, R20, R4, R5, R9: value (none) -> 0R2
- R23, R25: value (none) -> 1M
- R24, R26: value (none) -> 10k
- RN1: value (none) -> 1k; device resistor-dil:4R-NEXBS8V -> resistor-dil:4R-NCAT16
- U5: SPICEPREFIX (none) -> X
- U7: value ICL7660CPAZ -> ICL7660CPAZSOIC; device ICL7660CPAZ:ICL7660CPAZ -> ICL7660CPAZ:ICL7660CPAZSOIC
Connections:
- net N$1 renamed DAC_OUT
- net N$7 renamed AREF
- removed net N$12: SJ1.1, U3.AIN1
- removed net N$29: B1.+, C11.+, C12.+
- removed net VOLTAGE-: U3.AIN3
- new net +5V: SPI.2
- new net FAN: R30.1
- new net MISO: SPI.1, U4.PB4
- new net MOSI: SPI.4, U4.PB3
- new net N$1: Q7.B, R31.2, VR1.C
- new net N$30: Q6.G, R30.2
- new net N$38: R32.2, R33.1, VR1.R
- new net N$7: C11.+, C12.+, D1.C, D2.C, Q7.C, R31.1
- new net RST: SPI.5, U4.PC6/!RESET
- new net SCK: SPI.3, U4.PB5
- net -5V: now also C21.1
- net 12V: now also C26.+, IC7.IN, J2.1, Q7.E, R32.1, U$3.C; no longer IC2.VI
- net 4,5V: now also C24.+
- net 5V: now also C22.2, C23.1, C25.1, C27.+, IC7.OUT, IC7.OUT1, J3.3; no longer IC2.VO
- net CURRENT: now also RN1A.2, RN1B.2, RN1C.2, RN1D.2; no longer RN1A.1, RN1B.1, RN1C.1, RN1D.1
- net CURRENT1: now also RN1D.1; no longer RN1A.2
- net CURRENT2: now also RN1C.1; no longer RN1B.2
- net CURRENT3: now also RN1B.1; no longer RN1C.2
- net CURRENT4: now also RN1A.1; no longer RN1D.2
- net GND: now also C21.2, C22.1, C23.2, C24.-, C25.2, C26.-, C27.-, D3.A, D4.A, IC7.GND, J3.4, Q6.S, R33.2, SPI.6, U3.AIN3, VR1.A; no longer B1.-, IC2.GND, SJ1.2
- net N$24: now also J2.2, Q6.D, U$3.A; no longer R24.2, U5.OUT
- net N$25: now also J4.2; no longer J2.2
- net N$26: now also J4.1; no longer J2.1
- net N$27: now also D1.A, D3.C, J5.2; no longer B1.AC1, X1-1.KL
- net N$28: now also D2.A, D4.C, J5.1; no longer B1.AC2, X1-2.KL
- net SCL: now also J3.1
- net SDA: now also J3.2
- net VOLTAGE+: now also R24.2, U5.OUT
Other:
- note added: "Fan"
- note added: "I2C LCD"
- note added: "Input trigger"
- note added: "Power electronics"
- note added: "Programming connector"
- moved on the sheet: C1, C10, C11, C12, C16, C17, C19, C2, C20, C3, C4, C6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

Commit message: finished power supply, added keypad, programming connector, transient trigger and more
Parts:
- removed KK2: SK95-2M3, heatsink:SK95-2M3
- added C28, C29: 22p, rcl:C-EUC0603
- added D7: LL4148, diode:LL4148
- added J6, J7: B2B-XH-A(LF)(SN), JST_B2B-XH-A_LF__SN_:B2B-XH-A(LF)(SN)
- added JP1: (no value), pinhead:PINHD-1X7
- added JP2: (no value), pinhead:PINHD-1X4
- added Q10, Q11, Q8, Q9: MMBTA56-SOT23, transistor-pnp:MMBTA56-SOT23
- added Q12: CRYSTAL_3,4X2,7, CRYSTAL_SMD_3,4x2.7mm:CRYSTAL_3,4X2,7
- added R34, R35, R36: 10k, rcl:R-EU_R0603
- added R37, R38, R39, R40: 1k, rcl:R-EU_R0603
- added U$1: TO220_HEATSINK, custom_heatsink:TO220_HEATSINK
- added U8: PC817X2NIP0F, PC817X2NIP0F:PC817X2NIP0F
- R31: value 1R -> 100R
- R32, R33: value 1R -> 1k
- renumbered U$3 to D5
Connections:
- net N$1 renamed BASE
- net N$7 renamed 16V
- removed net +5V: SPI.2
- removed net MISO: SPI.1, U4.PB4
- removed net MOSI: SPI.4, U4.PB3
- new net KP1: JP1.1, U4.PD6
- new net KP2: JP1.2, U4.PD7
- new net KP3: JP1.3, U4.PB0
- new net KP4: JP1.4, U4.PB1
- new net KP5: JP1.5, U4.PB2
- new net KP6/MOSI: JP1.6, SPI.4, U4.PB3
- new net KP7/MISO: JP1.7, SPI.1, U4.PB4
- new net N$1: D7.K, R34.1, U8.A
- new net N$12: Q8.B, R37.2
- new net N$29: C28.1, Q12.1
- new net N$37: Q9.B, R38.2
- new net N$39: C29.1, Q12.3
- new net N$40: Q10.B, R39.2
- new net N$42: Q11.B, R40.2
- new net N$7: J7.2, R34.2
- new net OFF: R37.1, R38.1, R39.1, R40.1, U4.PD4
- new net RX: JP2.2, U4.PD0
- new net TEMP: J6.2, R35.2, U4.ADC6
- new net TRIGG: R36.1, U8.CT
- new net TX: JP2.3, U4.PD1
- new net XTL1: U4.PB6
- new net XTL2: U4.PB7
- net 5V: now also J6.1, Q10.E, Q11.E, Q8.E, Q9.E, R36.2, SPI.2
- net FAN: now also U4.PD5
- net GND: now also C28.2, C29.2, D7.A, J7.1, JP2.4, Q12.2, Q12.P$1, R35.1, U8.C, U8.ET
- net N$13: now also Q9.C
- net N$18: now also Q10.C
- net N$23: now also Q11.C
- net N$27: now also J5.1; no longer J5.2
- net N$28: now also J5.2; no longer J5.1
- net N$6: now also Q8.C
- net RST: now also JP2.1
Other:
- note added: "Addr: 0x60"
- note added: "Addr: 0x6f"
- note added: "Temperature measurement"
- note added: "Without C19, value of C17 and C18 is 10uF"
- note removed: "Addr: 0x60/0x61"
- moved on the sheet: C6, IC7, J5, SPI

Commit message: before voltage reference change
Parts:
- removed RN1: 1k, resistor-dil:4R-NCAT16
- added R41, R42, R43, R44: (no value), rcl:R-EU_R0603
- Q10, Q11, Q8, Q9: value MMBTA56-SOT23 -> S9015; device transistor-pnp:MMBTA56-SOT23 -> transistors:S9015
- Q5: value (none) -> 32768Hz
Connections:
- removed net N$29: C28.1, Q12.1
- removed net N$39: C29.1, Q12.3
- new net T_GND: D7.A, J7.1, U8.C
- net CURRENT: now also R41.1, R42.1, R43.1, R44.1; no longer RN1A.2, RN1B.2, RN1C.2, RN1D.2
- net CURRENT1: now also R44.2; no longer RN1D.1
- net CURRENT2: now also R43.2; no longer RN1C.1
- net CURRENT3: now also R42.2; no longer RN1B.1
- net CURRENT4: now also R41.2; no longer RN1A.1
- net GND: no longer D7.A, J7.1, U8.C
- net XTL1: now also C28.1, Q12.1
- net XTL2: now also C29.1, Q12.3
Other:
- note added: "Keypad"
- moved on the sheet: J6, JP1, R35

Commit message: new voltage reference
Parts:
- removed C10: 1u, rcl:C-EUC0805
- removed C20: 10u, rcl:C-EUC0805
- removed C24: 10u, rcl:CPOL-EUCT3528
- removed R29: 1R, rcl:R-EU_R0603
- removed U$2: REF5045IDSOIC, REF504x:REF5045IDSOIC
- added U$3: LM4140, voltage_references:LM4140
- C8: value 1u-10u -> 10u; device rcl:C-EUC0805 -> rcl:CPOL-EUCT3528
- C9: device rcl:C-EUC0805 -> rcl:CPOL-EUCT3216
- J2, J4, J5, J6, J7: value B2B-XH-A(LF)(SN) -> B2B-XH; device JST_B2B-XH-A_LF__SN_:B2B-XH-A(LF)(SN) -> jst connectors:B2B-XH
- J3: value B4B-XH-A(LF)(SN) -> B4B-XH; device B4B-XH-A_LF__SN_:B4B-XH-A(LF)(SN) -> jst connectors:B4B-XH
Connections:
- removed net 4,5V: C10.1, C13.1, C24.+, R27.1, R28.1, R29.2, U$2.VOUT, U2.VDD
- removed net N$19: C9.1, U$2.TRIM/NR
- removed net N$36: C20.1, R29.1
- new net 4,096V: C13.1, C9.+, R27.1, R28.1, U$3.VREF, U2.VDD
- net 5V: now also C8.+, U$3.ENABLE, U$3.VIN; no longer C8.1, U$2.VIN
- net GND: now also C8.-, C9.-, U$3.GND; no longer C10.2, C20.2, C24.-, C8.2, C9.2, U$2.GND

Commit message: finished V1.0
Parts:
- added J8: B5B-XH, jst connectors:B5B-XH
- added R29: 10k, rcl:R-EU_R0603
- C6: value (none) -> 100n
- JP2: value (none) -> B4B-XH; device pinhead:PINHD-1X4 -> jst connectors:B4B-XH
- R27, R28: value (none) -> 4k7
Connections:
- new net ENC_A: J8.3, U4.PD2
- new net ENC_B: J8.2, U4.PC3
- new net ENC_SW: J8.4, U4.PD3
- net 5V: now also J8.1, R29.1
- net GND: now also J8.5
- net RST: now also R29.2
- net TRIGG: now also U4.ADC7
Other:
- moved on the sheet: C6, R27, R28
