File: Electronic_load_PCB/Electronic_load.sch (EAGLE design)
At the start: 111 parts, among them IC7 LM1117IMPX-5.0, J1 XT60-M, J2 B2B-XH, J3 B4B-XH, J4 B2B-XH, J5 B2B-XH, J6 B2B-XH, J7 B2B-XH, J8 B5B-XH, Q1 IRFP250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

Commit message: changed some resistor values
Parts:
- R21: value 15k -> 10k
- R30: value 470R -> 1k
- R35: value 10k -> 47k
- R37, R38, R39, R40: value 1k -> 100k
Changed lines of the file:
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@@
 <part name="GND1" library="supply1" library_urn="urn:adsk.eagle:library:371" deviceset="GND" device=""/>
 <part name="VDD1" library="supply1" library_urn="urn:adsk.eagle:library:371" deviceset="VDD" device=""/>
-<part name="R21" library="rcl" library_urn="urn:adsk.eagle:library:334" deviceset="R-EU_" device="R0603" package3d_urn="urn:adsk.eagle:package:23555/3" value="15k"/>
+<part name="R21" library="rcl" library_urn="urn:adsk.eagle:library:334" deviceset="R-EU_" device="R0603" package3d_urn="urn:adsk.eagle:package:23555/3" value="10k"/>
 <part name="R22" library="rcl" library_urn="urn:adsk.eagle:library:334" deviceset="R-EU_" device="R0603" package3d_urn="urn:adsk.eagle:package:23555/3" value="1k"/>
 <part name="GND2" library="supply1" library_urn="urn:adsk.eagle:library:371" deviceset="GND" device=""/>
@@
 <part name="Q6" library="IRLML6244" deviceset="IRLML6244" device="" package3d_urn="urn:adsk.eagle:package:36516986/2"/>
 <part name="D5" library="BYG22B" deviceset="BYG22B" device="" package3d_urn="urn:adsk.eagle:package:43416/2"/>
-<part name="R30" library="rcl" library_urn="urn:adsk.eagle:library:334" deviceset="R-EU_" device="R0603" package3d_urn="urn:adsk.eagle:package:23555/3" value="470R"/>
+<part name="R30" library="rcl" library_urn="urn:adsk.eagle:library:334" deviceset="R-EU_" device="R0603" package3d_urn="urn:adsk.eagle:package:23555/3" value="1k"/>
 <part name="J3" library="jst connectors" deviceset="B4B-XH" device="" package3d_urn="urn:adsk.eagle:package:36544612/2"/>
 <part name="C23" library="rcl" library_urn="urn:adsk.eagle:library:334" deviceset="C-EU" device="C0603K" package3d_urn="urn:adsk.eagle:package:23680/2" value="100n"/>
@@
 <part name="U$1" library="custom_heatsink" deviceset="TO220_HEATSINK" device="" override_package3d_urn="urn:adsk.eagle:package:36629292/4" override_package_urn="urn:adsk.eagle:footprint:36629293/2"/>
 <part name="R34" library="rcl" library_urn="urn:adsk.eagle:library:334" deviceset="R-EU_" device="R0603" package3d_urn="urn:adsk.eagle:package:23555/3" value="10k"/>
-<part name="R35" library="rcl" library_urn="urn:adsk.eagle:library:334" deviceset="R-EU_" device="R0603" package3d_urn="urn:adsk.eagle:package:23555/3" value="10k"/>
+<part name="R35" library="rcl" library_urn="urn:adsk.eagle:library:334" deviceset="R-EU_" device="R0603" package3d_urn="urn:adsk.eagle:package:23555/3" value="47k"/>
 <part name="GND44" library="supply1" library_urn="urn:adsk.eagle:library:371" deviceset="GND" device=""/>
 <part name="VDD16" library="supply1" library_urn="urn:adsk.eagle:library:371" deviceset="VDD" device=""/>
@@
 <part name="Q8" library="transistors" deviceset="S9015" device="" override_package3d_urn="urn:adsk.eagle:package:36704401/2" override_package_urn="urn:adsk.eagle:footprint:20709/1"/>
 <part name="VDD29" library="supply1" library_urn="urn:adsk.eagle:library:371" deviceset="VDD" device=""/>
-<part name="R37" library="rcl" library_urn="urn:adsk.eagle:library:334" deviceset="R-EU_" device="R0603" package3d_urn="urn:adsk.eagle:package:23555/3" value="1k"/>
+<part name="R37" library="rcl" library_urn="urn:adsk.eagle:library:334" deviceset="R-EU_" device="R0603" package3d_urn="urn:adsk.eagle:package:23555/3" value="100k"/>
 <part name="Q9" library="transistors" deviceset="S9015" device="" override_package3d_urn="urn:adsk.eagle:package:36704402/2" override_package_urn="urn:adsk.eagle:footprint:20709/1"/>
 <part name="VDD26" library="supply1" library_urn="urn:adsk.eagle:library:371" deviceset="VDD" device=""/>
-<part name="R38" library="rcl" library_urn="urn:adsk.eagle:library:334" deviceset="R-EU_" device="R0603" package3d_urn="urn:adsk.eagle:package:23555/3" value="1k"/>
+<part name="R38" library="rcl" library_urn="urn:adsk.eagle:library:334" deviceset="R-EU_" device="R0603" package3d_urn="urn:adsk.eagle:package:23555/3" value="100k"/>
 <part name="Q10" library="transistors" deviceset="S9015" device="" override_package3d_urn="urn:adsk.eagle:package:36704403/2" override_package_urn="urn:adsk.eagle:footprint:20709/1"/>
 <part name="VDD27" library="supply1" library_urn="urn:adsk.eagle:library:371" deviceset="VDD" device=""/>
-<part name="R39" library="rcl" library_urn="urn:adsk.eagle:library:334" deviceset="R-EU_" device="R0603" package3d_urn="urn:adsk.eagle:package:23555/3" value="1k"/>
+<part name="R39" library="rcl" library_urn="urn:adsk.eagle:library:334" deviceset="R-EU_" device="R0603" package3d_urn="urn:adsk.eagle:package:23555/3" value="100k"/>
 <part name="Q11" library="transistors" deviceset="S9015" device="" override_package3d_urn="urn:adsk.eagle:package:36704397/2" override_package_urn="urn:adsk.eagle:footprint:20709/1"/>
 <part name="VDD28" library="supply1" library_urn="urn:adsk.eagle:library:371" deviceset="VDD" device=""/>
-<part name="R40" library="rcl" library_urn="urn:adsk.eagle:library:334" deviceset="R-EU_" device="R0603" package3d_urn="urn:adsk.eagle:package:23555/3" value="1k"/>
+<part name="R40" library="rcl" library_urn="urn:adsk.eagle:library:334" deviceset="R-EU_" device="R0603" package3d_urn="urn:adsk.eagle:package:23555/3" value="100k"/>
 <part name="D7" library="diode" deviceset="LL4148" device="" override_package3d_urn="urn:adsk.eagle:package:36704398/2" override_package_urn="urn:adsk.eagle:footprint:36704399/1"/>
 <part name="C28" library="rcl" library_urn="urn:adsk.eagle:library:334" deviceset="C-EU" device="C0603" package3d_urn="urn:adsk.eagle:package:23616/2" value="22p"/>

Commit message: cleaned up schematic
Parts:
- removed Q12: CRYSTAL_3,4X2,7, CRYSTAL_SMD_3,4x2.7mm:CRYSTAL_3,4X2,7
- added U$2: CRYSTAL_3,4X2,7, CRYSTAL_SMD_3,4x2.7mm:CRYSTAL_3,4X2,7
- C17, C18: value 100u -> 10u
- C19: value 100p -> omit
- C25: value 1u -> 100n
- R31: value 100R -> 1k
- R34: value 10k -> 1k
- R35: value 47k -> 10k
Connections:
- net GND: now also U$2.2; no longer Q12.2, Q12.P$1
- net XTL1: now also U$2.1; no longer Q12.1
- net XTL2: now also U$2.3; no longer Q12.3
Other:
- note added: "9th pin is for potential upgrade to a 4x5 keypad"
- note added: "Encoder"
- note added: "Programming connectors"
- note added: "The efficiency at low load can be increased by adding C19 which lowers the oscillator frequency"
- note added: "UART"
- note removed: "Programming connector"
- note removed: "Without C19, value of C17 and C18 is 10uF"
- moved on the sheet: C1, C11, C12, C13, C14, C15, C16, C17, C18, C19, C2, C21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
