File: pcb_front/Electronic_load_front_PCB.sch (EAGLE design)
At the start: 9 parts, among them SW1 EC12E_SW

Commit message: encoder works great, bounces reduced
Parts:
- added C1, C2, C3: 100n, rcl:C-EUC0603
- R1, R2: value (none) -> 4k7
- R3: value (none) -> 12k
Connections:
- net ENC_A: now also C2.1
- net ENC_B: now also C3.1
- net ENC_SW: now also C1.1
- net GND: now also C1.2, C2.2, C3.2
Other:
- moved on the sheet: JP1
Changed lines of the file:
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@@
 <part name="GND4" library="supply1" library_urn="urn:adsk.eagle:library:371" deviceset="GND" device=""/>
 <part name="P+1" library="supply1" library_urn="urn:adsk.eagle:library:371" deviceset="VCC" device=""/>
-<part name="R1" library="rcl" library_urn="urn:adsk.eagle:library:334" deviceset="R-EU_" device="R0603" package3d_urn="urn:adsk.eagle:package:23555/3"/>
-<part name="R2" library="rcl" library_urn="urn:adsk.eagle:library:334" deviceset="R-EU_" device="R0603" package3d_urn="urn:adsk.eagle:package:23555/3"/>
-<part name="R3" library="rcl" library_urn="urn:adsk.eagle:library:334" deviceset="R-EU_" device="R0603" package3d_urn="urn:adsk.eagle:package:23555/3"/>
+<part name="R1" library="rcl" library_urn="urn:adsk.eagle:library:334" deviceset="R-EU_" device="R0603" package3d_urn="urn:adsk.eagle:package:23555/3" value="4k7"/>
+<part name="R2" library="rcl" library_urn="urn:adsk.eagle:library:334" deviceset="R-EU_" device="R0603" package3d_urn="urn:adsk.eagle:package:23555/3" value="4k7"/>
+<part name="R3" library="rcl" library_urn="urn:adsk.eagle:library:334" deviceset="R-EU_" device="R0603" package3d_urn="urn:adsk.eagle:package:23555/3" value="12k"/>
 <part name="S1" library="switch" library_urn="urn:adsk.eagle:library:380" deviceset="TL46PO" device="" package3d_urn="urn:adsk.eagle:package:27746/1" override_package3d_urn="urn:adsk.eagle:package:36740710/2" override_package_urn="urn:adsk.eagle:footprint:27637/1"/>
 <part name="JP2" library="pinhead" library_urn="urn:adsk.eagle:library:325" deviceset="PINHD-1X2" device="/90" package3d_urn="urn:adsk.eagle:package:22437/2"/>
 <part name="JP3" library="pinhead" library_urn="urn:adsk.eagle:library:325" deviceset="PINHD-1X2" device="/90" package3d_urn="urn:adsk.eagle:package:22437/2"/>
 <part name="JP4" library="pinhead" library_urn="urn:adsk.eagle:library:325" deviceset="PINHD-1X2" device="/90" package3d_urn="urn:adsk.eagle:package:22437/2"/>
+<part name="C1" library="rcl" library_urn="urn:adsk.eagle:library:334" deviceset="C-EU" device="C0603" package3d_urn="urn:adsk.eagle:package:23616/2" value="100n"/>
+<part name="C2" library="rcl" library_urn="urn:adsk.eagle:library:334" deviceset="C-EU" device="C0603" package3d_urn="urn:adsk.eagle:package:23616/2" value="100n"/>
+<part name="C3" library="rcl" library_urn="urn:adsk.eagle:library:334" deviceset="C-EU" device="C0603" package3d_urn="urn:adsk.eagle:package:23616/2" value="100n"/>
+<part name="GND5" library="supply1" library_urn="urn:adsk.eagle:library:371" deviceset="GND" device=""/>
+<part name="GND6" library="supply1" library_urn="urn:adsk.eagle:library:371" deviceset="GND" device=""/>
+<part name="GND7" library="supply1" library_urn="urn:adsk.eagle:library:371" deviceset="GND" device=""/>
 </parts>
 <sheets>
@@
 <instance part="P+2" gate="VCC" x="22.86" y="76.2" smashed="yes"/>
 <instance part="P+3" gate="VCC" x="38.1" y="76.2" smashed="yes"/>
-<instance part="JP1" gate="A" x="-7.62" y="55.88" smashed="yes" rot="R180">
-<attribute name="NAME" x="-1.27" y="47.625" size="1.778" layer="95" rot="R180"/>
-<attribute name="VALUE" x="-1.27" y="66.04" size="1.778" layer="96" rot="R180"/>
-</instance>
-<instance part="GND4" gate="1" x="2.54" y="45.72" smashed="yes">
-<attribute name="VALUE" x="0" y="43.18" size="1.778" layer="96"/>
-</instance>
-<instance part="P+1" gate="VCC" x="2.54" y="66.04" smashed="yes"/>
+<instance part="JP1" gate="A" x="-20.32" y="55.88" smashed="yes" rot="R180">
+<attribute name="NAME" x="-13.97" y="47.625" size="1.778" layer="95" rot="R180"/>
+<attribute name="VALUE" x="-13.97" y="66.04" size="1.778" layer="96" rot="R180"/>
+</instance>
+<instance part="GND4" gate="1" x="-10.16" y="35.56" smashed="yes">
+<attribute name="VALUE" x="-12.7" y="33.02" size="1.778" layer="96"/>
+</instance>
+<instance part="P+1" gate="VCC" x="-10.16" y="66.04" smashed="yes"/>
 <instance part="R1" gate="G$1" x="17.78" y="66.04" smashed="yes" rot="R90">
 <attribute name="NAME" x="16.2814" y="62.23" size="1.778" layer="95" rot="R90"/>
@@
 <attribute name="NAME" x="70.485" y="67.31" size="1.778" layer="95" rot="R90"/>
 <attribute name="VALUE" x="81.28" y="67.31" size="1.778" layer="96" rot="R90"/>
+</instance>
+<instance part="C1" gate="G$1" x="12.7" y="45.72" smashed="yes">
+<attribute name="NAME" x="14.224" y="46.101" size="1.778" layer="95"/>
+<attribute name="VALUE" x="14.224" y="41.021" size="1.778" layer="96"/>
+</instance>
+<instance part="C2" gate="G$1" x="5.08" y="45.72" smashed="yes">
+<attribute name="NAME" x="6.604" y="46.101" size="1.778" layer="95"/>
+<attribute name="VALUE" x="6.604" y="41.021" size="1.778" layer="96"/>
+</instance>
+<instance part="C3" gate="G$1" x="-2.54" y="45.72" smashed="yes">
+<attribute name="NAME" x="-1.016" y="46.101" size="1.778" layer="95"/>
+<attribute name="VALUE" x="-1.016" y="41.021" size="1.778" layer="96"/>
+</instance>
+<instance part="GND5" gate="1" x="-2.54" y="35.56" smashed="yes">
+<attribute name="VALUE" x="-5.08" y="33.02" size="1.778" layer="96"/>
+</instance>
+<instance part="GND6" gate="1" x="5.08" y="35.56" smashed="yes">
+<attribute name="VALUE" x="2.54" y="33.02" size="1.778" layer="96"/>
+</instance>
+<instance part="GND7" gate="1" x="12.7" y="35.56" smashed="yes">
+<attribute name="VALUE" x="10.16" y="33.02" size="1.778" layer="96"/>
 </instance>
 </instances>
@@
 <pinref part="JP1" gate="A" pin="1"/>
 <pinref part="GND4" gate="1" pin="GND"/>
-<wire x1="-5.08" y1="50.8" x2="2.54" y2="50.8" width="0.1524" layer="91"/>
-<wire x1="2.54" y1="50.8" x2="2.54" y2="48.26" width="0.1524" layer="91"/>
+<wire x1="-17.78" y1="50.8" x2="-10.16" y2="50.8" width="0.1524" layer="91"/>
+<wire x1="-10.16" y1="50.8" x2="-10.16" y2="38.1" width="0.1524" layer="91"/>
+</segment>
+<segment>
+<pinref part="C3" gate="G$1" pin="2"/>
+<pinref part="GND5" gate="1" pin="GND"/>
+<wire x1="-2.54" y1="40.64" x2="-2.54" y2="38.1" width="0.1524" layer="91"/>
+</segment>
+<segment>
+<pinref part="C2" gate="G$1" pin="2"/>
+<pinref part="GND6" gate="1" pin="GND"/>
+<wire x1="5.08" y1="40.64" x2="5.08" y2="38.1" width="0.1524" layer="91"/>
+</segment>
+<segment>
+<pinref part="C1" gate="G$1" pin="2"/>
+<pinref part="GND7" gate="1" pin="GND"/>
+<wire x1="12.7" y1="40.64" x2="12.7" y2="38.1" width="0.1524" layer="91"/>
 </segment>
 </net>
@@
 <segment>
 <pinref part="JP1" gate="A" pin="5"/>
-<wire x1="-5.08" y1="60.96" x2="2.54" y2="60.96" width="0.1524" layer="91"/>
+<wire x1="-17.78" y1="60.96" x2="-10.16" y2="60.96" width="0.1524" layer="91"/>
 <pinref part="P+1" gate="VCC" pin="VCC"/>
-<wire x1="2.54" y1="60.96" x2="2.54" y2="63.5" width="0.1524" layer="91"/>
-<label x="5.08" y="68.58" size="1.778" layer="95" rot="R180"/>
+<wire x1="-10.16" y1="60.96" x2="-10.16" y2="63.5" width="0.1524" layer="91"/>
+<label x="-7.62" y="68.58" size="1.778" layer="95" rot="R180"/>
 </segment>
 </net>
@@
 <wire x1="38.1" y1="60.96" x2="38.1" y2="53.34" width="0.1524" layer="91"/>
 <wire x1="38.1" y1="53.34" x2="38.1" y2="50.8" width="0.1524" layer="91"/>
-<wire x1="-5.08" y1="53.34" x2="38.1" y2="53.34" width="0.1524" layer="91"/>
+<wire x1="-17.78" y1="53.34" x2="12.7" y2="53.34" width="0.1524" layer="91"/>
 <junction x="38.1" y="53.34"/>
+<pinref part="C1" gate="G$1" pin="1"/>
+<wire x1="12.7" y1="53.34" x2="38.1" y2="53.34" width="0.1524" layer="91"/>
+<wire x1="12.7" y1="48.26" x2="12.7" y2="53.34" width="0.1524" layer="91"/>
+<junction x="12.7" y="53.34"/>
 </segment>
 </net>
@@
 <wire x1="25.4" y1="60.96" x2="25.4" y2="55.88" width="0.1524" layer="91"/>
 <wire x1="25.4" y1="55.88" x2="25.4" y2="50.8" width="0.1524" layer="91"/>
-<wire x1="-5.08" y1="55.88" x2="25.4" y2="55.88" width="0.1524" layer="91"/>
+<wire x1="-17.78" y1="55.88" x2="5.08" y2="55.88" width="0.1524" layer="91"/>
 <junction x="25.4" y="55.88"/>
+<pinref part="C2" gate="G$1" pin="1"/>
+<wire x1="5.08" y1="55.88" x2="25.4" y2="55.88" width="0.1524" layer="91"/>
+<wire x1="5.08" y1="48.26" x2="5.08" y2="55.88" width="0.1524" layer="91"/>
+<junction x="5.08" y="55.88"/>
 </segment>
 </net>
@@
 <wire x1="20.32" y1="60.96" x2="20.32" y2="58.42" width="0.1524" layer="91"/>
 <wire x1="20.32" y1="58.42" x2="20.32" y2="50.8" width="0.1524" layer="91"/>
-<wire x1="-5.08" y1="58.42" x2="20.32" y2="58.42" width="0.1524" layer="91"/>
+<wire x1="-17.78" y1="58.42" x2="-2.54" y2="58.42" width="0.1524" layer="91"/>
 <junction x="20.32" y="58.42"/>
-</segment>
-</net>
+<pinref part="C3" gate="G$1" pin="1"/>
+<wire x1="-2.54" y1="58.42" x2="20.32" y2="58.42" width="0.1524" layer="91"/>
+<wire x1="-2.54" y1="48.26" x2="-2.54" y2="58.42" width="0.1524" layer="91"/>
+<junction x="-2.54" y="58.42"/>
+</segment>
+</net>
