File: pcb_main/Electronic_load.brd (EAGLE design)
At the start: 121.9 x 88.6 mm, 111 parts, among them IC7 LM1117IMPX-5.0, J1 XT60-M, J2 B2B-XH, J3 B4B-XH, J4 B2B-XH, J5 B2B-XH, J6 B2B-XH, J7 B2B-XH, J8 B5B-XH, Q1 IRFP250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

Commit message: added C10, schematic minor updates
Parts:
- added C10: 1u, rcl:C0603
Connections:
- net BASE: now also C10.1
- net GND: now also C10.2
Routing:
- net BASE: track 10.2 -> 12.3 mm
Changed lines of the file:
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@@
 <drawing>
 <settings>
-<setting alwaysvectorfont="no"/>
+<setting alwaysvectorfont="yes"/>
 <setting verticaltext="up"/>
 </settings>
@@
 <param name="mdViaViaSameLayer" value="6mil"/>
 <param name="mnLayersViaInSmd" value="2"/>
-<param name="mdCopperDimension" value="0mil"/>
+<param name="mdCopperDimension" value="1mil"/>
 <param name="mdDrill" value="6mil"/>
 <param name="mdSmdStop" value="0mil"/>
@@
 <attribute name="MF" value="Sharp Microelectronics" x="83.82" y="6.985" size="1.778" layer="27" display="off"/>
 <attribute name="MP" value="PC817X2NIP0F" x="83.82" y="6.985" size="1.778" layer="27" display="off"/>
+<attribute name="NAME" x="81.01816875" y="10.08701875" size="1.27083125" layer="25"/>
 <attribute name="NAME" x="81.014759375" y="10.0908" size="1.27238125" layer="25"/>
-<attribute name="NAME" x="81.01816875" y="10.08701875" size="1.27083125" layer="25"/>
 <attribute name="PACKAGE" value="SMD-4 Sharp" x="83.82" y="6.985" size="1.778" layer="27" display="off"/>
 <attribute name="PRICE" value="None" x="83.82" y="6.985" size="1.778" layer="27" display="off"/>
@@
 </element>
 <element name="U$2" library="CRYSTAL_SMD_3,4x2.7mm" package="CRYSTAL_3,4X2,7" value="CRYSTAL_3,4X2,7" x="101.6" y="11.43" smashed="yes" rot="MR270"/>
+<element name="C10" library="rcl" library_urn="urn:adsk.eagle:library:334" package="C0603" package3d_urn="urn:adsk.eagle:package:23616/2" value="1u" x="32.385" y="20.32" smashed="yes" rot="MR90">
+<attribute name="NAME" x="33.401" y="19.05" size="1.016" layer="26" rot="MR90"/>
+<attribute name="POPULARITY" value="73" x="32.385" y="20.32" size="1.778" layer="28" rot="MR90" display="off"/>
+<attribute name="SPICEPREFIX" value="C" x="32.385" y="20.32" size="1.778" layer="28" rot="MR90" display="off"/>
+<attribute name="VALUE" x="30.48" y="19.685" size="1.27" layer="28" rot="MR90"/>
+</element>
 </elements>
 <signals>
@@
 <contactref element="U$2" pad="GND"/>
 <contactref element="U$2" pad="GND2"/>
+<contactref element="C10" pad="2"/>
 </signal>
 <signal name="DAC_OUT">
@@
 <wire x1="30.48" y1="15.875" x2="31.75" y2="14.605" width="0.4064" layer="1"/>
 <wire x1="31.75" y1="14.605" x2="31.75" y2="12.7" width="0.4064" layer="1"/>
+<contactref element="C10" pad="1"/>
+<wire x1="32.385" y1="19.47" x2="31.75" y2="19.47" width="0.3048" layer="16"/>
+<wire x1="31.75" y1="19.47" x2="31.33" y2="19.05" width="0.3048" layer="16"/>
+<wire x1="31.33" y1="19.05" x2="30.48" y2="19.05" width="0.3048" layer="16"/>
 </signal>
 <signal name="N$38">
