File: pcb_main/Electronic_load.sch (EAGLE design)
At the start: 111 parts, among them IC7 LM1117IMPX-5.0, J1 XT60-M, J2 B2B-XH, J3 B4B-XH, J4 B2B-XH, J5 B2B-XH, J6 B2B-XH, J7 B2B-XH, J8 B5B-XH, Q1 IRFP250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

Commit message: added C10, schematic minor updates
Parts:
- added C10: 1u, rcl:C-EUC0603
Connections:
- net BASE: now also C10.1
- net GND: now also C10.2
Other:
- note added: "Note: desolder pull-up resistors on LCD I2C module"
