File: pcb/pcb_front/Electronic_load_front_PCB.brd (EAGLE design)
At the start: 33 x 46.7 mm, 12 parts, among them SW1 EC12E_SW

Commit message: cleanup
Parts:
- JP1: device pinhead:1X05/90 -> pinhead:1X05
- moved JP1 3.81 mm to (5.08, 31.8)
Routing:
- net ENC_B: track 30.5 -> 33.5 mm
- net N$5: track 39.1 -> 40.7 mm
Other:
- outline, holes or cut-outs redrawn
Changed lines of the file:
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@@
 <setting verticaltext="up"/>
 </settings>
-<grid distance="50" unitdist="mil" unit="mil" style="lines" multiple="1" display="no" altdistance="5" altunitdist="mil" altunit="mil"/>
+<grid distance="25" unitdist="mil" unit="mil" style="lines" multiple="1" display="no" altdistance="5" altunitdist="mil" altunit="mil"/>
 <layers>
 <layer number="1" name="Top" color="4" fill="1" visible="yes" active="yes"/>
@@
 </layers>
 <board>
-<fusionsync huburn="a.YnVzaW5lc3M6Z21haWw1MzQ2MjM" projecturn="a.YnVzaW5lc3M6Z21haWw1MzQ2MjMjRDIwMTkxMjI5MjUwNjU0MjU2" f3durn="urn:adsk.wipprod:dm.lineage:3ZborseaTM63qMjKJInqhQ" pcbguid="" lastpulledtime="" lastsyncedchangeguid="" latestrevisionid="de9a6022-fa4f-43a6-98fc-7768da42b81b" lastsyncedrevisionid="de9a6022-fa4f-43a6-98fc-7768da42b81b" lastboardhashguid="187d4fe6-ef17-b919-9e19-ddac4a4cb30f" lastpushedtime="2022-08-03T22:12:43Z" linktopcb3d="false"/>
+<fusionsync huburn="a.YnVzaW5lc3M6Z21haWw1MzQ2MjM" projecturn="a.YnVzaW5lc3M6Z21haWw1MzQ2MjMjRDIwMTkxMjI5MjUwNjU0MjU2" f3durn="urn:adsk.wipprod:dm.lineage:3ZborseaTM63qMjKJInqhQ" pcbguid="" lastpulledtime="" lastsyncedchangeguid="" latestrevisionid="de9a6022-fa4f-43a6-98fc-7768da42b81b" lastsyncedrevisionid="de9a6022-fa4f-43a6-98fc-7768da42b81b" lastboardhashguid="187d4fe6-ef17-b919-9e19-ddac4a4cb30f" lastpushedtime="2022-08-03T22:12:43Z" linktopcb3d="true"/>
 <plain>
-<wire x1="0" y1="0" x2="33" y2="0" width="0" layer="20"/>
-<wire x1="33" y1="0" x2="33" y2="46.66" width="0" layer="20"/>
-<wire x1="33" y1="46.66" x2="0" y2="46.66" width="0" layer="20"/>
-<wire x1="0" y1="46.66" x2="0" y2="0" width="0" layer="20"/>
+<wire x1="0" y1="44.12" x2="0" y2="2.54" width="0" layer="20"/>
+<wire x1="0" y1="2.54" x2="2.54" y2="0" width="0" layer="20" curve="90"/>
+<wire x1="2.54" y1="0" x2="30.46" y2="0" width="0" layer="20"/>
+<wire x1="30.46" y1="0" x2="33" y2="2.54" width="0" layer="20" curve="90"/>
+<wire x1="33" y1="2.54" x2="33" y2="44.12" width="0" layer="20"/>
+<wire x1="33" y1="44.12" x2="30.46" y2="46.66" width="0" layer="20" curve="90"/>
+<wire x1="30.46" y1="46.66" x2="2.54" y2="46.66" width="0" layer="20"/>
+<wire x1="2.54" y1="46.66" x2="0" y2="44.12" width="0" layer="20" curve="90"/>
 <circle x="20.32" y="33.02" radius="12.951509375" width="0.0762" layer="47"/>
 <circle x="2.77" y="2.77" radius="1.5" width="0.0762" layer="20"/>
@@
 <attribute name="VALUE" x="16.82" y="42.02" size="1.27" layer="27"/>
 </element>
-<element name="JP1" library="pinhead" library_urn="urn:adsk.eagle:library:325" package="1X05/90" package3d_urn="urn:adsk.eagle:package:22467/2" value="" x="1.27" y="31.75" smashed="yes" rot="R90">
-<attribute name="NAME" x="8.2042" y="26.5938" size="1.27" layer="25" ratio="10" rot="R90"/>
-<attribute name="POPULARITY" value="9" x="1.27" y="31.75" size="1.778" layer="27" rot="R90" display="off"/>
-<attribute name="VALUE" x="4.445" y="25.4" size="1.27" layer="27" rot="R90"/>
+<element name="JP1" library="pinhead" library_urn="urn:adsk.eagle:library:325" package="1X05" package3d_urn="urn:adsk.eagle:package:22469/2" value="" x="5.08" y="31.75" smashed="yes" rot="R90">
+<attribute name="NAME" x="12.0142" y="26.5938" size="1.27" layer="25" ratio="10" rot="R90"/>
+<attribute name="POPULARITY" value="69" x="5.08" y="31.75" size="1.778" layer="27" rot="R90" display="off"/>
+<attribute name="VALUE" x="8.255" y="25.4" size="1.27" layer="27" rot="R90"/>
 </element>
 <element name="R1" library="rcl" library_urn="urn:adsk.eagle:library:334" package="R0603" package3d_urn="urn:adsk.eagle:package:23555/3" value="4k7" x="8.89" y="34.29" smashed="yes" rot="MR180">
@@
 <contactref element="SW1" pad="B"/>
 <wire x1="8.04" y1="31.75" x2="5.08" y2="31.75" width="0.6096" layer="16"/>
-<wire x1="5.08" y1="31.75" x2="4.191" y2="31.75" width="0.6096" layer="16"/>
-<wire x1="4.191" y1="31.75" x2="1.397" y2="34.544" width="0.6096" layer="16"/>
+<wire x1="5.08" y1="31.75" x2="4.064" y2="31.75" width="0.6096" layer="16"/>
+<wire x1="4.064" y1="31.75" x2="1.397" y2="34.417" width="0.6096" layer="16"/>
 <wire x1="1.397" y1="38.869" x2="3.048" y2="40.52" width="0.6096" layer="16"/>
 <wire x1="3.048" y1="40.52" x2="13.97" y2="40.52" width="0.6096" layer="16"/>
 <wire x1="13.97" y1="40.52" x2="17.82" y2="40.52" width="0.6096" layer="16"/>
-<wire x1="1.397" y1="34.544" x2="1.397" y2="38.869" width="0.6096" layer="16"/>
+<wire x1="1.397" y1="34.417" x2="1.397" y2="38.869" width="0.6096" layer="16"/>
 <contactref element="C2" pad="1"/>
 <wire x1="13.97" y1="41.06" x2="13.97" y2="40.52" width="0.6096" layer="16"/>
@@
 <contactref element="SW1" pad="A"/>
 <wire x1="5.08" y1="34.29" x2="8.04" y2="34.29" width="0.6096" layer="16"/>
-<wire x1="5.08" y1="34.29" x2="4.9911" y2="34.3789" width="0.6096" layer="16"/>
-<wire x1="4.9911" y1="34.3789" x2="3.81" y2="34.417" width="0.6096" layer="16"/>
+<wire x1="5.08" y1="34.29" x2="6.61221875" y2="34.32660625" width="0.6096" layer="16"/>
+<wire x1="6.61221875" y1="34.32660625" x2="3.81" y2="34.417" width="0.6096" layer="16"/>
 <wire x1="3.81" y1="34.417" x2="2.667" y2="35.56" width="0.6096" layer="16"/>
 <wire x1="2.667" y1="35.56" x2="2.667" y2="37.719" width="0.6096" layer="16"/>
@@
 <contactref element="S1" pad="5"/>
 <contactref element="JP2" pad="1"/>
-<wire x1="5.08" y1="13.97" x2="4.826" y2="13.97" width="0.6096" layer="16"/>
-<wire x1="4.826" y1="13.97" x2="2.667" y2="11.811" width="0.6096" layer="16"/>
+<wire x1="5.08" y1="13.97" x2="3.556" y2="13.97" width="0.6096" layer="16"/>
+<wire x1="3.556" y1="13.97" x2="2.032" y2="12.446" width="0.6096" layer="16"/>
 <wire x1="10.414" y1="1.651" x2="23.368" y2="1.651" width="0.6096" layer="16"/>
 <wire x1="23.368" y1="1.651" x2="24.892" y2="3.175" width="0.6096" layer="16"/>
@@
 <wire x1="24.892" y1="6.477" x2="23.749" y2="7.62" width="0.6096" layer="16"/>
 <wire x1="23.749" y1="7.62" x2="22.86" y2="7.62" width="0.6096" layer="16"/>
-<wire x1="2.667" y1="6.858" x2="3.683" y2="5.842" width="0.6096" layer="16"/>
-<wire x1="3.683" y1="5.842" x2="6.223" y2="5.842" width="0.6096" layer="16"/>
+<wire x1="2.032" y1="6.858" x2="3.048" y2="5.842" width="0.6096" layer="16"/>
+<wire x1="3.048" y1="5.842" x2="6.223" y2="5.842" width="0.6096" layer="16"/>
 <wire x1="6.223" y1="5.842" x2="10.414" y2="1.651" width="0.6096" layer="16"/>
-<wire x1="2.667" y1="11.811" x2="2.667" y2="6.858" width="0.6096" layer="16"/>
+<wire x1="2.032" y1="12.446" x2="2.032" y2="6.858" width="0.6096" layer="16"/>
 </signal>
 <signal name="N$7">
@@
 <mfgpreviewcolor name="soldermaskcolor" color="0xC8000000"/>
 <mfgpreviewcolor name="silkscreencolor" color="0xFFFEFEFE"/>
-<mfgpreviewcolor name="backgroundcolor" color="0xFF282828"/>
+<mfgpreviewcolor name="backgroundcolor" color="0xFFFF0000"/>
 <mfgpreviewcolor name="coppercolor" color="0xFFC6C6C6"/>
 <mfgpreviewcolor name="substratecolor" color="0xFF786E46"/>
