File: pcb/pcb_front/front_board.brd (EAGLE design)
At the start: 33 x 46.7 mm, 12 parts, among them SW1 EC12E_SW

Commit message: cleanup
Parts:
- JP1: device pinhead:1X05 -> pinhead:1X05/90
- moved JP2 6.35 mm to (1.27, 21.6)
- moved JP4 6.35 mm to (1.27, 15.2)
- moved JP1 3.81 mm to (1.27, 31.8)
Connections:
- net N$1: now also JP4.2; no longer JP2.2
- net N$5: now also JP4.1; no longer JP2.1
- net N$8: now also JP2.1; no longer JP4.1
- net N$9: now also JP2.2; no longer JP4.2
Routing:
- net ENC_B: track 33.5 -> 31.0 mm
Other:
- board text added: "5V"
- board text added: "A"
- board text added: "B"
- board text added: "Electronic load Front board V1.1 Dominik Workshop 27.03.2024"
- board text added: "GND"
- board text added: "Main terminals"
- board text added: "Remote sense"
- board text added: "SW"
- board text added: "Voltage measure"
- board text removed: "V in"
- board text removed: "V sense in"
- board text removed: "V sense out"
