File: pcb/pcb_front/front_board.sch (EAGLE design)
At the start: 12 parts, among them SW1 EC12E_SW

Commit message: cleanup
Parts:
- JP1: device pinhead:PINHD-1X5 -> pinhead:PINHD-1X5/90
Connections:
- net N$1: now also JP4.2; no longer JP2.2
- net N$5: now also JP4.1; no longer JP2.1
- net N$8: now also JP2.1; no longer JP4.1
- net N$9: now also JP2.2; no longer JP4.2
Other:
- note added: "Dominik Wokshop"
- note added: "Electronic load front board"
- moved on the sheet: JP2, JP4
Changed lines of the file:
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@@
 <setting verticaltext="up"/>
 </settings>
-<grid distance="0.1" unitdist="inch" unit="inch" style="lines" multiple="1" display="no" altdistance="0.05" altunitdist="inch" altunit="inch"/>
+<grid distance="0.1" unitdist="inch" unit="inch" style="lines" multiple="1" display="no" altdistance="0.01" altunitdist="inch" altunit="inch"/>
 <layers>
 <layer number="1" name="Top" color="4" fill="1" visible="no" active="no"/>
@@
 <part name="P+2" library="supply1" library_urn="urn:adsk.eagle:library:371" deviceset="VCC" device=""/>
 <part name="P+3" library="supply1" library_urn="urn:adsk.eagle:library:371" deviceset="VCC" device=""/>
-<part name="JP1" library="pinhead" library_urn="urn:adsk.eagle:library:325" deviceset="PINHD-1X5" device="" package3d_urn="urn:adsk.eagle:package:22469/2"/>
+<part name="JP1" library="pinhead" library_urn="urn:adsk.eagle:library:325" deviceset="PINHD-1X5" device="/90" package3d_urn="urn:adsk.eagle:package:22467/2"/>
 <part name="GND4" library="supply1" library_urn="urn:adsk.eagle:library:371" deviceset="GND" device=""/>
 <part name="P+1" library="supply1" library_urn="urn:adsk.eagle:library:371" deviceset="VCC" device=""/>
@@
 <part name="R3" library="rcl" library_urn="urn:adsk.eagle:library:334" deviceset="R-EU_" device="R0603" package3d_urn="urn:adsk.eagle:package:23555/3" value="12k"/>
 <part name="S1" library="switch" library_urn="urn:adsk.eagle:library:380" deviceset="TL46PO" device="" package3d_urn="urn:adsk.eagle:package:27746/1" override_package3d_urn="urn:adsk.eagle:package:36740710/2" override_package_urn="urn:adsk.eagle:footprint:27637/1"/>
+<part name="JP4" library="pinhead" library_urn="urn:adsk.eagle:library:325" deviceset="PINHD-1X2" device="/90" package3d_urn="urn:adsk.eagle:package:22437/2"/>
+<part name="JP3" library="pinhead" library_urn="urn:adsk.eagle:library:325" deviceset="PINHD-1X2" device="/90" package3d_urn="urn:adsk.eagle:package:22437/2"/>
 <part name="JP2" library="pinhead" library_urn="urn:adsk.eagle:library:325" deviceset="PINHD-1X2" device="/90" package3d_urn="urn:adsk.eagle:package:22437/2"/>
-<part name="JP3" library="pinhead" library_urn="urn:adsk.eagle:library:325" deviceset="PINHD-1X2" device="/90" package3d_urn="urn:adsk.eagle:package:22437/2"/>
-<part name="JP4" library="pinhead" library_urn="urn:adsk.eagle:library:325" deviceset="PINHD-1X2" device="/90" package3d_urn="urn:adsk.eagle:package:22437/2"/>
 <part name="C1" library="rcl" library_urn="urn:adsk.eagle:library:334" deviceset="C-EU" device="C0603" package3d_urn="urn:adsk.eagle:package:23616/2" value="100n"/>
 <part name="C2" library="rcl" library_urn="urn:adsk.eagle:library:334" deviceset="C-EU" device="C0603" package3d_urn="urn:adsk.eagle:package:23616/2" value="100n"/>
@@
 <text x="115.57" y="40.64" size="1.778" layer="97">Voltage
 measure</text>
+<text x="93.98" y="10.16" size="3.81" layer="94">Electronic load
+front board</text>
+<text x="140.97" y="20.32" size="2.54" layer="94">Dominik Wokshop</text>
 </plain>
 <instances>
@@
 <attribute name="NAME" x="96.52" y="53.34" size="1.778" layer="95" rot="R180"/>
 </instance>
-<instance part="JP2" gate="G$1" x="111.76" y="41.91" smashed="yes">
+<instance part="JP4" gate="G$1" x="111.76" y="41.91" smashed="yes">
 <attribute name="NAME" x="105.41" y="47.625" size="1.778" layer="95"/>
 <attribute name="VALUE" x="105.41" y="36.83" size="1.778" layer="96"/>
@@
 <attribute name="VALUE" x="80.01" y="30.48" size="1.778" layer="96" rot="MR0"/>
 </instance>
-<instance part="JP4" gate="G$1" x="73.66" y="50.8" smashed="yes" rot="R180">
+<instance part="JP2" gate="G$1" x="73.66" y="50.8" smashed="yes" rot="R180">
 <attribute name="NAME" x="80.01" y="45.085" size="1.778" layer="95" rot="R180"/>
 <attribute name="VALUE" x="80.01" y="55.88" size="1.778" layer="96" rot="R180"/>
@@
 <wire x1="93.98" y1="86.36" x2="93.98" y2="91.44" width="0.1524" layer="91"/>
 <junction x="93.98" y="91.44"/>
+<label x="70.612" y="91.948" size="1.27" layer="95"/>
 </segment>
 </net>
@@
 <wire x1="86.36" y1="86.36" x2="86.36" y2="93.98" width="0.1524" layer="91"/>
 <junction x="86.36" y="93.98"/>
+<label x="70.612" y="94.488" size="1.27" layer="95"/>
 </segment>
 </net>
@@
 <wire x1="78.74" y1="86.36" x2="78.74" y2="96.52" width="0.1524" layer="91"/>
 <junction x="78.74" y="96.52"/>
+<label x="70.612" y="97.028" size="1.27" layer="95"/>
 </segment>
 </net>
@@
 <wire x1="99.06" y1="38.1" x2="101.6" y2="38.1" width="0.1524" layer="91"/>
 <wire x1="101.6" y1="38.1" x2="101.6" y2="41.91" width="0.1524" layer="91"/>
-<pinref part="JP2" gate="G$1" pin="2"/>
+<pinref part="JP4" gate="G$1" pin="2"/>
 <wire x1="101.6" y1="41.91" x2="109.22" y2="41.91" width="0.1524" layer="91"/>
 </segment>
@@
 <wire x1="99.06" y1="48.26" x2="101.6" y2="48.26" width="0.1524" layer="91"/>
 <wire x1="101.6" y1="48.26" x2="101.6" y2="44.45" width="0.1524" layer="91"/>
-<pinref part="JP2" gate="G$1" pin="1"/>
+<pinref part="JP4" gate="G$1" pin="1"/>
 <wire x1="101.6" y1="44.45" x2="109.22" y2="44.45" width="0.1524" layer="91"/>
 </segment>
@@
 <net name="N$8" class="0">
 <segment>
-<pinref part="JP4" gate="G$1" pin="1"/>
+<pinref part="JP2" gate="G$1" pin="1"/>
 <wire x1="76.2" y1="48.26" x2="86.36" y2="48.26" width="0.1524" layer="91"/>
 <wire x1="86.36" y1="48.26" x2="86.36" y2="40.64" width="0.1524" layer="91"/>
@@
 <net name="N$9" class="0">
 <segment>
-<pinref part="JP4" gate="G$1" pin="2"/>
+<pinref part="JP2" gate="G$1" pin="2"/>
 <pinref part="S1" gate="BEF1" pin="S1"/>
 <wire x1="76.2" y1="50.8" x2="88.9" y2="50.8" width="0.1524" layer="91"/>
